Commit message: Add physical manipulation and navigation scenes
Model accessory collision geometry and separate self-collision proxies from environment contact. Add shared task scenes and strengthen robot model validation.

File: urdf/franka_tmr.xacro (robot description, xacro)
@@ -245,4 +245,10 @@
         </material>
       </visual>
+      <collision>
+        <origin rpy="${pi/2} 0 ${pi/2}" />
+        <geometry>
+          <cylinder radius="${height}" length="${height*1.5}" />
+        </geometry>
+      </collision>
       <inertial>
         <origin xyz="-0.000344 -0.021232 0.038239" rpy="0 0 0"/>

File: urdf/imu.xacro (robot description, xacro)
@@ -4,4 +4,5 @@
     <link name="${prefix}imu_link">
       <visual><geometry><box size="0.03 0.03 0.01"/></geometry></visual>
+      <collision><geometry><box size="0.03 0.03 0.01"/></geometry></collision>
     </link>
     <joint name="${prefix}imu_joint" type="fixed">

File: urdf/mfr3duo.urdf (robot description, URDF)
Before this commit: robot mfr3duo, 134 links, 133 joints
Links:
- link front_realsense_d455_link: geometry collision mesh filename=package://mfr3duo_description/urdf/meshes/realsense_d455/vi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 scale=0.001 0.001 0.001; visual mesh filename=package://mfr3duo_description/urdf/meshes/realsense_d455/vi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 scale=0.001 0.001 0.001
- link head_zed_mini_link: geometry collision mesh filename=package://mfr3duo_description/urdf/meshes/zed_mini/visual/z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; visual mesh filename=package://mfr3duo_description/urdf/meshes/zed_mini/visual/z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
- link imu_imu_link: geometry collision box size=0.03 0.03 0.01; visual box size=0.03 0.03 0.01
- link left_d435_link: geometry collision mesh filename=package://mfr3duo_description/urdf/meshes/realsense_d435/vi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; visual mesh filename=package://mfr3duo_description/urdf/meshes/realsense_d435/vi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
- link left_wrist_camera_mount_link: geometry collision mesh filename=package://mfr3duo_description/urdf/meshes/wrist_camera_moun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 scale=0.001 0.001 0.001; visual mesh filename=package://mfr3duo_description/urdf/meshes/wrist_camera_moun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 scale=0.001 0.001 0.001
- link lidar_front_nanoscan3_link: geometry collision mesh filename=package://mfr3duo_description/urdf/meshes/nanoscan3/visual/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; visual mesh filename=package://mfr3duo_description/urdf/meshes/nanoscan3/visual/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
- link lidar_rear_nanoscan3_link: geometry collision mesh filename=package://mfr3duo_description/urdf/meshes/nanoscan3/visual/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; visual mesh filename=package://mfr3duo_description/urdf/meshes/nanoscan3/visual/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
- link rear_realsense_d455_link: geometry collision mesh filename=package://mfr3duo_description/urdf/meshes/realsense_d455/vi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 scale=0.001 0.001 0.001; visual mesh filename=package://mfr3duo_description/urdf/meshes/realsense_d455/vi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 scale=0.001 0.001 0.001
- link right_d435_link: geometry collision mesh filename=package://mfr3duo_description/urdf/meshes/realsense_d435/vi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; visual mesh filename=package://mfr3duo_description/urdf/meshes/realsense_d435/vi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
- link right_wrist_camera_mount_link: geometry collision mesh filename=package://mfr3duo_description/urdf/meshes/wrist_camera_moun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 scale=0.001 0.001 0.001; visual mesh filename=package://mfr3duo_description/urdf/meshes/wrist_camera_moun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 scale=0.001 0.001 0.001
- link rocker_arm_link: geometry collision cylinder length=0.0225 radius=0.015; visual cylinder length=0.0225 radius=0.015

File: urdf/nanoscan3.xacro (robot description, xacro)
@@ -8,4 +8,8 @@
         <material name="mfr3duo_sensor_dark_gray"/>
       </visual>
+      <collision>
+        <origin xyz="-0.01 -0.08 -0.04" rpy="0 0 ${pi/2}"/>
+        <geometry><mesh filename="package://mfr3duo_description/urdf/meshes/nanoscan3/visual/NANS3.dae"/></geometry>
+      </collision>
     </link>
     <joint name="${prefix}nanoscan3_joint" type="fixed">

File: urdf/realsense_d435.xacro (robot description, xacro)
@@ -13,4 +13,8 @@
         <material name="mfr3duo_sensor_aluminum"/>
       </visual>
+      <collision>
+        <origin xyz="0.0043 -0.0175 0" rpy="${pi/2} 0 ${pi/2}"/>
+        <geometry><mesh filename="package://mfr3duo_description/urdf/meshes/realsense_d435/visual/d435.dae"/></geometry>
+      </collision>
     </link>
     <joint name="${prefix}d435_joint" type="fixed">

File: urdf/realsense_d455.xacro (robot description, xacro)
@@ -8,4 +8,8 @@
         <material name="mfr3duo_sensor_aluminum"/>
       </visual>
+      <collision>
+        <origin xyz="0.00465 -0.0475 0" rpy="${pi/2} 0 ${pi/2}"/>
+        <geometry><mesh filename="package://mfr3duo_description/urdf/meshes/realsense_d455/visual/d455.stl" scale="0.001 0.001 0.001"/></geometry>
+      </collision>
     </link>
     <joint name="${prefix}realsense_d455_joint" type="fixed">

File: urdf/wrist_camera_mount.xacro (robot description, xacro)
@@ -8,4 +8,8 @@
         <material name="mfr3duo_printed_mount"/>
       </visual>
+      <collision>
+        <origin xyz="-0.024 -0.03 0"/>
+        <geometry><mesh filename="package://mfr3duo_description/urdf/meshes/wrist_camera_mount/visual/RealSenseD435_Camera_Mount.stl" scale="0.001 0.001 0.001"/></geometry>
+      </collision>
     </link>
     <joint name="${prefix}wrist_camera_mount_joint" type="fixed">

File: urdf/zed_mini.xacro (robot description, xacro)
@@ -7,4 +7,7 @@
         <material name="mfr3duo_sensor_black"/>
       </visual>
+      <collision>
+        <geometry><mesh filename="package://mfr3duo_description/urdf/meshes/zed_mini/visual/zedm.stl"/></geometry>
+      </collision>
     </link>
     <joint name="${prefix}zed_mini_joint" type="fixed">
